File: hardware/EchoSafe_RevA/EchoSafe_RevA/EchoSafe_RevA.kicad_pcb (KiCad board)
At the start: 2 copper layers, 260 x 175 mm, 29 parts, among them J1 TP4056_Module, J2 Conn_Harness_09, J3 Conn_Harness_09, J4 Conn_Harness_07, J5 Conn_Harness_07, U1 ESP32-S3-WROOM-1-N16R8, U2 MAX98357AETE+T, U3 DRV2605LDGS, U5 TCA9548A, U6 DRV2605LDGS, U7 DRV2605LDGS, U8 DRV2605LDGS

Commit message: Fix TP4056 module footprint shape, sync R2/J1 changes to PCB
The TP4056 J1 footprint was a generic uniform-pitch 4-pin header, which
research (product photos + two independently-measured same-family
boards) shows is the wrong shape entirely -- the real module has all 4
pins in a single column with uneven spacing. Replaced with a custom
footprint built from that data (TP4056_Module.pretty), flagged as a
best estimate pending physical confirmation.

Also synced the schematic's R2 (TCA9548A RESET pull-up) and the new J1
footprint through to the actual PCB layout, which hadn't been touched
since those schematic edits -- rerouted the affected nets around the
existing copper. Verified via kicad-cli pcb drc: 0 violations, 0
unconnected pads.

Co-Authored-By: Claude Sonnet 5 <noreply@anthropic.com>
Parts:
- added R2: 10k, R_0603_1608Metric, F.Cu at (65.0, 83.0)
- J1: footprint PinHeader_1x04_P2.54mm_Vertical -> TP4056_Module
- moved J1 8.56 mm to (45.0, 3.44)
Connections:
- U5 pad 3: 3V3_SYS -> TCA_RESET
Routing:
- net TCA_RESET: track 0.00 -> 26.0 mm
- net VSYS: track 49.6 -> 63.2 mm, vias 0 -> 2
- net 3V3_SYS: track 558.3 -> 568.9 mm
- net VBAT: track 26.2 -> 31.3 mm
- net GND: track 790.3 -> 788.8 mm

Commit message: Resize central pod from 260x175mm to a compact 65x90mm
The previous DRC-driven routing (hand-written attempts + FreeRouting)
had no board-size constraint, leaving the central pod tablet-sized
despite being fully DRC-clean -- not remotely wearable-scale. Re-placed
all 22 components into a logical floorplan sized from real component
extents (front/rear harness connectors on opposite edges, power/
charging cluster on one side for access, MCU centered, haptic driver
cluster below it), then re-routed via FreeRouting from scratch.

Routed clean in a single pass this time: 0 unrouted, 0 violations,
score 999.99/1000, confirmed independently via kicad-cli pcb drc (0
violations, 0 unconnected pads). Traces came out at 0.15-0.2mm
throughout, within standard fab capability.

Still not ready to order: acoustic port holes on the mic modules,
a visual review, physical TP4056 footprint confirmation, and fab
outputs (gerbers/BOM/CPL) -- none generated yet.

Co-Authored-By: Claude Sonnet 5 <noreply@anthropic.com>
Parts:
- moved J3 164.0 mm to (44.0, 8.00)
- moved J2 161.8 mm to (16.0, 8.00)
- moved J5 145.6 mm to (44.0, 80.0)
- moved C17 143.9 mm to (11.0, 24.0)
- moved C15 141.4 mm to (11.0, 20.0)
- moved J4 136.2 mm to (16.0, 80.0)
- moved C18 123.5 mm to (11.0, 34.0)
- moved R1 119.9 mm to (11.0, 30.0)
- moved C14 115.4 mm to (36.0, 68.0)
- moved C7 110.4 mm to (10.0, 58.0)
- moved C13 109.5 mm to (36.0, 50.0)
- moved U2 105.3 mm to (30.0, 68.0)
- moved U7 102.3 mm to (15.0, 58.0)
- moved U8 98.2 mm to (45.0, 58.0)
- moved C8 96.0 mm to (50.0, 62.0)
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Routing:
- net GND: track 788.8 -> 368.2 mm, vias 12 -> 2
- net 3V3_SYS: track 568.9 -> 326.3 mm, vias 10 -> 7
- net SPK_OUTN: track 307.1 -> 101.6 mm, vias 2 -> 3
- net MUX_CH3_SDA: track 150.3 -> 19.2 mm
- net MUX_CH3_SCL: track 145.5 -> 20.1 mm
- net MIC_TOP_WS: track 182.5 -> 64.4 mm, vias 5 -> 4
- net MIC_TOP_SCK: track 168.0 -> 57.8 mm, vias 4 -> 3
- net MUX_CH2_SCL: track 129.0 -> 20.3 mm
- net MUX_CH2_SDA: track 133.8 -> 34.4 mm, vias 2 -> 6
- net SPK_OUTP: track 200.6 -> 102.5 mm
- net MIC_TOP_SD: track 167.4 -> 70.3 mm, vias 6 -> 3
- net MUX_CH1_SDA: track 117.3 -> 20.3 mm
- net MUX_CH1_SCL: track 112.5 -> 19.0 mm
- net MIC_BOT_SD: track 170.0 -> 79.1 mm, vias 2 -> 3
- net MUX_CH0_SDA: track 100.8 -> 16.3 mm
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Other:
- board size 260 x 175 mm -> 65 x 90 mm

Commit message: Visual/silkscreen review: fix footprint FPID prefixes and silkscreen overlaps
kicad-cli pcb drc was only ever run at default severity, which silently
excludes the silk_over_copper/silk_overlap/text_height checks. Re-running
with --severity-all, plus rendering true F.SilkS-only SVGs (previous
renders mixed in F.Fab assembly-doc text, making boards look far more
cluttered than they are), surfaced real issues:

- Every placed footprint on all 5 boards had lost its library prefix
  (bare name, no "Library:" qualifier) despite correct fp-lib-table
  registrations -- pcbnew's Python API doesn't preserve FPID library
  nicknames across a FootprintLoad()/board.Add() round-trip unless
  SetFPID() is called explicitly. Fixed across all 5 boards.
- The custom TP4056_Module footprint had its pads listing F.SilkS in
  their own layer set (guaranteed self-violation on every pad) and
  center-justified pin labels straddling the outline/pad edges. Fixed
  in the library footprint and re-synced onto the central pod.
- H1 (acoustic port) and M1 (motor) reference text overlapped MIC1's
  pads and undersized text vs. the board's minimum, respectively --
  fixed in their library footprints and re-synced onto all 4 modules.
- U2's reference sat on its own QFN thermal pad; C8's reference
  overlapped neighboring C4's silkscreen; U1/U2 each carried a literal
  duplicate coincident silkscreen text object (UltraLibrarian import
  artifact). All fixed.

All 5 boards now show 0 DRC violations at full severity (previously
only verified at default severity). Two items flagged but left
unfixed since they'd require hand-editing KiCad's own shared global
library footprints: J1/LS1 connectors have no pin-1 marker on the
physically-printed silkscreen (only on F.Fab), and U1's reference
will be hidden under the soldered ESP32 module.

Co-Authored-By: Claude Sonnet 5 <noreply@anthropic.com>
Parts:
- BT1: footprint JST_PH_S2B-PH-K_1x02_P2.00mm_Horizontal -> Connector_JST:JST_PH_S2B-PH-K_1x02_P2.00mm_Horizontal
- C1, C13, C14, C15, C16, C17, C18, C2, C3, C4, C5, C6, C7, C8: footprint C_0603_1608Metric -> Capacitor_SMD:C_0603_1608Metric
- J1: footprint TP4056_Module -> TP4056_Module:TP4056_Module
- J2, J3: footprint JST_SH_SM09B-SRSS-TB_1x09-1MP_P1.00mm_Horizontal -> Connector_JST:JST_SH_SM09B-SRSS-TB_1x09-1MP_P1.00mm_Horizontal
- J4, J5: footprint JST_SH_SM07B-SRSS-TB_1x07-1MP_P1.00mm_Horizontal -> Connector_JST:JST_SH_SM07B-SRSS-TB_1x07-1MP_P1.00mm_Horizontal
- LD1: footprint PinHeader_1x03_P2.54mm_Vertical -> Connector_PinHeader_2.54mm:PinHeader_1x03_P2.54mm_Vertical
- R1, R2: footprint R_0603_1608Metric -> Resistor_SMD:R_0603_1608Metric
- U1: footprint ESP32-S3-WROOM-1_EXP -> ESP32-S3-WROOM-1:ESP32-S3-WROOM-1_EXP
- U2: footprint 21-0136I_T1633-4_MXM -> MAX98357AETE-T:21-0136I_T1633-4_MXM
- U3, U6, U7, U8: footprint VSSOP-10_3x3mm_P0.5mm -> Package_SO:VSSOP-10_3x3mm_P0.5mm
- U5: footprint TSSOP-24_4.4x7.8mm_P0.65mm -> Package_SO:TSSOP-24_4.4x7.8mm_P0.65mm

Commit message: Add pin-1 silkscreen markers and relocate U1's hidden reference
Follow-up to the visual/silkscreen review: both previously-flagged
items are now addressed.

- J1 (all 4 modules + central pod J2-J5) and LS1 (front modules) used
  KiCad's stock Connector_JST/Connector_Molex footprints, whose F.SilkS
  pin-1 indicator is only a subtle asymmetric notch in the outline
  (easy to miss at this scale) -- not, as first described, entirely
  absent. Rather than hand-edit KiCad's shared global libraries, added
  a project-local override library (lib/symbols/Connectors_PinMarked.pretty)
  with a bold pin-1 dot added to each of the 3 affected footprints, and
  resynced every affected instance onto it.
- U1 (ESP32-S3-WROOM-1)'s reference sat inside the module's own
  footprint outline (hidden once the module is soldered down).
  Checked every neighboring footprint and routed trace via pcbnew's
  Python API to see if it could move outside the outline into open
  board area -- it can't; this board was deliberately packed to a
  minimum practical 65x90mm and nothing borders U1 with room to spare.
  Moved the reference within the footprint's own interior instead, to
  a pocket clear of the trace and secondary pad cluster it previously
  sat on top of -- fully legible pre-assembly, same as before post-
  assembly (matches the original "cosmetic only" assessment).

All 5 boards re-verified at 0 DRC violations, full severity.

Co-Authored-By: Claude Sonnet 5 <noreply@anthropic.com>
Parts:
- J2, J3: value Conn_Harness_09 -> JST_SH_SM09B-SRSS-TB_1x09-1MP_P1.00mm_Horizontal; footprint Connector_JST:JST_SH_SM09B-SRSS-TB_1x09-1MP_P1.00mm_Horizontal -> Connectors_PinMarked:JST_SH_SM09B-SRSS-TB_1x09-1MP_P1.00mm_Horizontal
- J4, J5: value Conn_Harness_07 -> JST_SH_SM07B-SRSS-TB_1x07-1MP_P1.00mm_Horizontal; footprint Connector_JST:JST_SH_SM07B-SRSS-TB_1x07-1MP_P1.00mm_Horizontal -> Connectors_PinMarked:JST_SH_SM07B-SRSS-TB_1x07-1MP_P1.00mm_Horizontal
