File: hardware/EchoSafe_RevA/EchoSafe_RevA/EchoSafe_RevA.kicad_sch (KiCad schematic)
At the start: 30 parts, among them J1 TP4056_Module, J2 Conn_Harness_09, J3 Conn_Harness_09, J4 Conn_Harness_07, J5 Conn_Harness_07, U1 ESP32-S3-WROOM-1-N16R8, U2 MAX98357AETE+T, U3 DRV2605LDGS, U5 TCA9548A, U6 DRV2605LDGS, U7 DRV2605LDGS, U8 DRV2605LDGS

Commit message: Fix TP4056 module footprint shape, sync R2/J1 changes to PCB
The TP4056 J1 footprint was a generic uniform-pitch 4-pin header, which
research (product photos + two independently-measured same-family
boards) shows is the wrong shape entirely -- the real module has all 4
pins in a single column with uneven spacing. Replaced with a custom
footprint built from that data (TP4056_Module.pretty), flagged as a
best estimate pending physical confirmation.

Also synced the schematic's R2 (TCA9548A RESET pull-up) and the new J1
footprint through to the actual PCB layout, which hadn't been touched
since those schematic edits -- rerouted the affected nets around the
existing copper. Verified via kicad-cli pcb drc: 0 violations, 0
unconnected pads.

Co-Authored-By: Claude Sonnet 5 <noreply@anthropic.com>
Parts:
- J1: footprint Connector_PinHeader_2.54mm:PinHeader_1x04_P2.54mm_Vertical -> TP4056_Module:TP4056_Module
Changed lines of the file:
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@@
 			(effects (font (size 1.27 1.27)) (justify left))
 		)
-		(property "Footprint" "Connector_PinHeader_2.54mm:PinHeader_1x04_P2.54mm_Vertical"
+		(property "Footprint" "TP4056_Module:TP4056_Module"
 			(at 190 10 0)
 			(effects (font (size 1.27 1.27) (italic yes)) (hide yes))
@@
 			(effects (font (size 1.27 1.27)) (hide yes))
 		)
-		(property "Description" "HiLetGo TP4056 Li-ion charger module w/ protection"
+		(property "Description" "HiLetGo TP4056 Li-ion charger module w/ protection -- footprint pin spacing is a best estimate from research (not the physical board), see CLAUDE.md"
 			(at 190 10 0)
 			(effects (font (size 1.27 1.27)) (hide yes))

Commit message: Generate fab outputs (gerbers, drill, CPL, BOM) for all 5 boards
kicad-cli pcb export gerbers/drill/pos and sch export bom, into each
project's own outputs/ folder, zipped for direct fab upload. Standard
2-layer gerber set (confirmed 2-layer by checking the layer table, not
assumed); drill files split PTH/NPTH since the mic modules have a real
NPTH hole (H1, the acoustic port) -- spot-checked the NPTH file directly
to confirm it's really in there.

Generating the BOM surfaced a real gap: J2/J3/J4/J5 (central pod), J1
(all 4 modules), and LS1 (front modules) still had their schematic
Footprint field pointing at the stock Connector_JST/Connector_Molex
footprint, not the Connectors_PinMarked override from the last commit --
because that fix only touched footprint instances already placed on the
PCB, never the originating schematic symbols. Left alone, a future
"Update PCB from Schematic" would have silently reverted the pin-marker
fix. Fixed by updating the Footprint property in each .kicad_sch;
confirmed via kicad-cli sch erc that violation counts on all 5 schematics
are unchanged (metadata-only edit, no electrical effect).

All 5 boards reconfirmed at 0 DRC violations, full severity.

Co-Authored-By: Claude Sonnet 5 <noreply@anthropic.com>
Parts:
- J2, J3: footprint Connector_JST:JST_SH_SM09B-SRSS-TB_1x09-1MP_P1.00mm_Horizontal -> Connectors_PinMarked:JST_SH_SM09B-SRSS-TB_1x09-1MP_P1.00mm_Horizontal
- J4, J5: footprint Connector_JST:JST_SH_SM07B-SRSS-TB_1x07-1MP_P1.00mm_Horizontal -> Connectors_PinMarked:JST_SH_SM07B-SRSS-TB_1x07-1MP_P1.00mm_Horizontal
Changed lines of the file:
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@@
 			(effects (font (size 1.27 1.27)) (justify left))
 		)
-		(property "Footprint" "Connector_JST:JST_SH_SM09B-SRSS-TB_1x09-1MP_P1.00mm_Horizontal"
+		(property "Footprint" "Connectors_PinMarked:JST_SH_SM09B-SRSS-TB_1x09-1MP_P1.00mm_Horizontal"
 			(at 30 195 0)
 			(effects (font (size 1.27 1.27) (italic yes)) (hide yes))
@@
 			(effects (font (size 1.27 1.27)) (justify left))
 		)
-		(property "Footprint" "Connector_JST:JST_SH_SM09B-SRSS-TB_1x09-1MP_P1.00mm_Horizontal"
+		(property "Footprint" "Connectors_PinMarked:JST_SH_SM09B-SRSS-TB_1x09-1MP_P1.00mm_Horizontal"
 			(at 70 195 0)
 			(effects (font (size 1.27 1.27) (italic yes)) (hide yes))
@@
 			(effects (font (size 1.27 1.27)) (justify left))
 		)
-		(property "Footprint" "Connector_JST:JST_SH_SM07B-SRSS-TB_1x07-1MP_P1.00mm_Horizontal"
+		(property "Footprint" "Connectors_PinMarked:JST_SH_SM07B-SRSS-TB_1x07-1MP_P1.00mm_Horizontal"
 			(at 110 195 0)
 			(effects (font (size 1.27 1.27) (italic yes)) (hide yes))
@@
 			(effects (font (size 1.27 1.27)) (justify left))
 		)
-		(property "Footprint" "Connector_JST:JST_SH_SM07B-SRSS-TB_1x07-1MP_P1.00mm_Horizontal"
+		(property "Footprint" "Connectors_PinMarked:JST_SH_SM07B-SRSS-TB_1x07-1MP_P1.00mm_Horizontal"
 			(at 250 195 0)
 			(effects (font (size 1.27 1.27) (italic yes)) (hide yes))
